File: rpizero-lowpower.sch (KiCad schematic (older format))
At the start: 39 parts, among them J1 Screw_Terminal_01x06, J2 Screw_Terminal_01x04, J3 Raspberry_Pi_2_3, J4 Conn_01x03, Q1 NDP6020, U1 ATtiny1604-SS

Commit message: bom updated with mouser part numbers
Parts:
- removed BT1: 3V7, myparts:18650-ebay, symbol Device:Battery_Cell
- removed H1, H2, H3, H4: MountingHole, myparts:MountingHole_5.3mm__no_courtyard, symbol Mechanical:MountingHole
- removed J1: Screw_Terminal_01x06, Connector_PinHeader_2.54mm:PinHeader_2x03_P2.54mm_Vertical, symbol Connector_Generic:Conn_01x06
- removed J2: Screw_Terminal_01x04, Connector_PinHeader_2.54mm:PinHeader_2x03_P2.54mm_Vertical, symbol Connector_Generic:Conn_01x06
- removed J3: Raspberry_Pi_2_3, myparts:Raspberry_Pi_Zero_Socketed_THT_FaceDown_MountingHoles_no_court, symbol Connector:Raspberry_Pi_2_3
- removed J4: Conn_01x03, Connector_PinHeader_2.54mm:PinHeader_1x03_P2.54mm_Vertical, symbol Connector_Generic:Conn_01x03
- C1, C2, C4, C6, C9: Vendor (none) -> 963-UMK212BJ104KG-T
- C3, C5, C7, C8: value 1u -> 100n; Vendor (none) -> 963-UMK212BJ104KG-T
- D1: Vendor (none) -> 607-CMDA5AR7D1S
- IO0, IO1, IO2, IO3, R1: Vendor (none) -> 603-RT0805FRE0710KL
- Q1: Vendor (none) -> 512-NDP6020P
- R10, R11, R12, R2, R7, R8, R9: Vendor (none) -> 603-RT0805FRE071KL
- R13, R5: Vendor (none) -> 284-APC0805B100KN
- R14: Vendor (none) -> 756-PCF0805R200KBI
- R3, R4: value 4k7 -> 10k; Vendor (none) -> 603-RT0805FRE0710KL
- R6: Vendor (none) -> 756-PCF0805R-90K9BT1
- U1: Vendor (none) -> 579-ATTINY1604-SSNR
